Commit message: Added ros2_control files and updated the launch file

File: autoport_bot/description/robot.urdf.xacro (robot description, xacro)
@@ -2,5 +2,6 @@
 <robot xmlns:xacro="http://www.ros.org/wiki/xacro"  name="robot">
     <xacro:include filename="robot_core.xacro"/>
-    <xacro:include filename="gazebo_control.xacro"/>
+    <!-- <xacro:include filename="gazebo_control.xacro"/> -->
     <xacro:include filename="lidar.xacro"/>
+    <xacro:include filename="ros2_control.xacro"/>
 </robot>

File: autoport_bot/description/robot_core.xacro (robot description, xacro)
@@ -25,4 +25,12 @@
         <origin xyz="-0.063 0 0"/>
     </joint>
+    <!--BASE FOOTPRINT LINK-->
+    <joint name="base_footprint_joint" type="fixed">
+        <parent link="base_link"/>
+        <child link="base_footprint"/>
+        <origin xyz = "0 0 0" rpy="0 0 0"/>
+    </joint>
+    <link name="base_footprint">
+    </link>
     <!--CHASSIS LINK-->
     <link name="chassis">
@@ -51,5 +59,5 @@
         <parent link = "base_link"/>
         <child link = "left_wheel"/>
-        <origin xyz="0 0.105 0" rpy="-${pi/2} 0 0"/>
+        <origin xyz="0 0.095 0" rpy="-${pi/2} 0 0"/>
         <axis xyz="0 0 1"/>
     </joint>
@@ -57,5 +65,5 @@
         <visual>
             <geometry>
-                <cylinder radius="0.037" length="0.022"/>
+                <cylinder radius="0.0355" length="0.021"/>
             </geometry>
             <material name ="blue"/>
@@ -63,8 +71,8 @@
         <collision>
             <geometry>
-                <cylinder radius="0.037" length="0.022"/>
+                <sphere radius="0.0355"/>
             </geometry>
         </collision>
-        <xacro:inertial_cylinder mass = "0.075" length="0.022" radius="0.037">
+        <xacro:inertial_cylinder mass = "0.075" length="0.021" radius="0.0355">
             <origin xyz="0 0 0" rpy="0 0 0"/>
         </xacro:inertial_cylinder>
@@ -77,5 +85,5 @@
         <parent link = "base_link"/>
         <child link = "right_wheel"/>
-        <origin xyz="0 -0.105 0" rpy="${pi/2} 0 0"/>
+        <origin xyz="0 -0.095 0" rpy="${pi/2} 0 0"/>
         <axis xyz="0 0 -1"/>
     </joint>
@@ -83,5 +91,5 @@
         <visual>
             <geometry>
-                <cylinder radius="0.037" length="0.022"/>
+                <cylinder radius="0.0355" length="0.021"/>
             </geometry>
             <material name ="blue"/>
@@ -89,8 +97,8 @@
         <collision>
             <geometry>
-                <cylinder radius="0.037" length="0.022"/>
+                <sphere radius="0.0355"/>
             </geometry>
         </collision>
-        <xacro:inertial_cylinder mass = "0.075" length="0.022" radius="0.037">
+        <xacro:inertial_cylinder mass = "0.075" length="0.021" radius="0.0355">
             <origin xyz="0 0 0" rpy="0 0 0"/>
         </xacro:inertial_cylinder>
