Commit message: Fixed serial port issue

File: autoport_bot/description/robot_core.xacro (robot description, xacro)
@@ -60,5 +60,5 @@
         <child link = "left_wheel"/>
         <origin xyz="0 0.095 0" rpy="-${pi/2} 0 0"/>
-        <axis xyz="0 0 1"/>
+        <axis xyz="0 0 -1"/>
     </joint>
     <link name = "left_wheel">

File: autoport_bot/description/ros2_control.xacro (robot description, xacro)
@@ -7,5 +7,5 @@
             <param name="right_wheel_name">right_wheel_joint</param>
             <param name="loop_rate">30</param>
-            <param name="device">/dev/ttyUSB1</param>
+            <param name="device">/dev/ttyUSB0</param>
             <param name="baud_rate">57600</param>
             <param name="timeout_ms">1000</param>
