Commit message: Create LICENSE
Changed Lidar library

Delete folder rplidar_ros

File: autoport_bot/description/lidar.xacro (robot description, xacro)
@@ -4,5 +4,6 @@
         <parent link="chassis"/>
         <child link="laser_frame"/>
-        <origin xyz="0.1 0 0.175" rpy="0 0 0"/>
+        <!-- originally laser_frame -->
+        <origin xyz="0.1 0 0.105" rpy="0 0 0"/>
     </joint>
     <link name = "laser_frame">

File: autoport_bot/description/robot_core.xacro (robot description, xacro)
@@ -20,9 +20,4 @@
     <link name="base_link">
     </link>
-    <joint name = "chassis_joint" type="fixed">
-        <parent link="base_link"/>
-        <child link="chassis"/>
-        <origin xyz="-0.063 0 0"/>
-    </joint>
     <!--BASE FOOTPRINT LINK-->
     <joint name="base_footprint_joint" type="fixed">
@@ -34,4 +29,9 @@
     </link>
     <!--CHASSIS LINK-->
+    <joint name = "chassis_joint" type="fixed">
+        <parent link="base_link"/>
+        <child link="chassis"/>
+        <origin xyz="-0.063 0 0"/>
+    </joint>
     <link name="chassis">
         <visual>
@@ -60,5 +60,5 @@
         <child link = "left_wheel"/>
         <origin xyz="0 0.095 0" rpy="-${pi/2} 0 0"/>
-        <axis xyz="0 0 -1"/>
+        <axis xyz="0 0 1"/>
     </joint>
     <link name = "left_wheel">
